Commit message: added gazebo launch

File: leg_assembly/urdf/leg_assembly.urdf (robot description, URDF)
Before this commit: robot leg_assembly, 10 links, 9 joints
Links:
- link base_link: geometry collision mesh filename=file://$(find leg_assembly)/meshes/base_link.STL; visual mesh filename=file://$(find leg_assembly)/meshes/base_link.STL
- link end_effector: geometry collision mesh filename=file://$(find leg_assembly)/meshes/end_effector.STL; visual mesh filename=file://$(find leg_assembly)/meshes/end_effector.STL
- link finger_link_left: geometry collision mesh filename=file://$(find leg_assembly)/meshes/finger_link_left.STL; visual mesh filename=file://$(find leg_assembly)/meshes/finger_link_left.STL
- link finger_link_right: geometry collision mesh filename=file://$(find leg_assembly)/meshes/finger_link_right.STL; visual mesh filename=file://$(find leg_assembly)/meshes/finger_link_right.STL
- link finger_tip_left: geometry collision mesh filename=file://$(find leg_assembly)/meshes/finger_tip_left.STL; visual mesh filename=file://$(find leg_assembly)/meshes/finger_tip_left.STL
- link finger_tip_right: geometry collision mesh filename=file://$(find leg_assembly)/meshes/finger_tip_right.STL; visual mesh filename=file://$(find leg_assembly)/meshes/finger_tip_right.STL
- link link_1: geometry collision mesh filename=file://$(find leg_assembly)/meshes/link_1.STL; visual mesh filename=file://$(find leg_assembly)/meshes/link_1.STL
- link link_2: geometry collision mesh filename=file://$(find leg_assembly)/meshes/link_2.STL; visual mesh filename=file://$(find leg_assembly)/meshes/link_2.STL
- link link_3: geometry collision mesh filename=file://$(find leg_assembly)/meshes/link_3.STL; visual mesh filename=file://$(find leg_assembly)/meshes/link_3.STL
- link link_4: geometry collision mesh filename=file://$(find leg_assembly)/meshes/link_4.STL; visual mesh filename=file://$(find leg_assembly)/meshes/link_4.STL

File: leg_assembly_moveit_config/config/gazebo_ros2_control.xacro (robot description, xacro)
@@ -1,10 +1,10 @@
 <?xml version="1.0"?>
 <robot xmlns:xacro="http://www.ros.org/wiki/xacro">
-    <xacro:macro name="leg_assembly_ros2_control" params="name initial_positions_file">
-        <xacro:property name="initial_positions" value="${load_yaml(initial_positions_file)['initial_positions']}"/>
+    <xacro:macro name="gazebo_ros2_control" params="name initial_positions_file">
+        <xacro:property name="initial_positions" value="${xacro.load_yaml(initial_positions_file)['initial_positions']}"/>
         <ros2_control name="${name}" type="system">
             <hardware>
                 <!-- By default, set up controllers for simulation. This won't work on real hardware -->
-                <plugin>mock_components/GenericSystem</plugin>
+                <plugin>gazebo_ros2_control/GazeboSystem</plugin>
             </hardware>
             <joint name="base_joint">
